File: KiCad files/AGB-E06-10.kicad_pcb (KiCad board)
At the start: 2 copper layers, 51 x 30.8 mm, 21 parts, among them U0 CartBus, U1 MX23L12806-12C, U2 FM18W08-SG

Commit message: Add files via upload
Routing:
- net A15: track 26.2 -> 22.6 mm
- net A14: track 70.1 -> 66.5 mm
- net CS: track 38.3 -> 37.6 mm
- net A7: track 77.5 -> 78.1 mm
- net A3: track 61.9 -> 61.3 mm
